Commit message: Updated rviz, modified params

File: urdf/udacity_bot_new.xacro (robot description, xacro)
@@ -138,8 +138,36 @@
         <joint_properties damping="1.0" friction="1.0"/>
    </joint>
+   <link name="body">
+     <inertial>
+        <mass value="0.1"/>
+        <origin xyz="-0.05 0 0.1" rpy=" 0 0 0"/>
+        <inertia
+            ixx="1e-6" ixy="0" ixz="0"
+            iyy="1e-6" iyz="0" izz="1e-6"
+        />
+      </inertial>
+      <collision name='collision'>
+        <origin xyz="-0.05 0 0.1" rpy=" 0 0 0"/>
+        <geometry>
+          <box size="0.1 0.1 0.3"/>
+        </geometry>
+      </collision>
+      <visual name='chassis_visual'>
+        <origin xyz="-0.05 0 0.1" rpy=" 0 0 0"/>
+        <geometry>
+           <box size="0.15 0.15 0.3"/>
+        </geometry>
+      </visual>
+     </link>
+     <joint type="fixed" name="body_joint">
+          <origin xyz="-0.05 0 0" rpy="0 0 0"/>
+          <parent link="chassis"/>
+          <child link="body"/>
+          <axis xyz="0 1 0" rpy="0 0 0"/>
+     </joint>
  <link name="camera">
    <inertial>
       <mass value="0.1"/>
-      <origin xyz="0 0 0" rpy=" 0 0 0"/>
+      <origin xyz="-0.05 0 0.14" rpy=" 0 0 0"/>
       <inertia
           ixx="1e-6" ixy="0" ixz="0"
@@ -148,18 +176,18 @@
     </inertial>
     <collision name='collision'>
-      <origin xyz="0 0 0" rpy=" 0 0 0"/>
-      <geometry>
-        <box size="0.05 0.05 0.05"/>
-      </geometry>
-    </collision>
-    <visual name='chassis_visual'>
-      <origin xyz="0 0 0" rpy=" 0 0 0"/>
-      <geometry>
-         <box size="0.05 0.05 0.05"/>
+      <origin xyz="-0.05 0 0.14" rpy=" 0 0 0"/>
+      <geometry>
+        <box size="0.06 0.06 0.06"/>
+      </geometry>
+    </collision>
+    <visual name='chassis_visual'>
+      <origin xyz="-0.05 0 0.14" rpy=" 0 0 0"/>
+      <geometry>
+         <box size="0.06 0.06 0.06"/>
       </geometry>
     </visual>
    </link>
    <joint type="fixed" name="camera_joint">
-        <origin xyz="0.2 0 0" rpy="0 0 0"/>
+        <origin xyz="-0.05 0 0.14" rpy="0 0 0"/>
         <parent link="chassis"/>
         <child link="camera"/>
